File: Placa/TCC.sch (EAGLE design)
At the start: 98 parts, among them IC1 LM324N, IC2 MEGA8-P, IC3 788TV, IC6 LM324N, IC7 LM741P, Q2 BC548, Q3 IRFI540NPBF, Q4 IRFI540NPBF, Q5 IRFI540NPBF, Q6 IRFI540NPBF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

Commit message: Signed-off-by: Jéfferson Pimenta Melo <jefferson.pimenta@hotmail.com>
Parts:
- C10, C11, C15, C16, C17, C18, C21, C22, C25: value (none) -> 10uF
- C12, C20, C23, C24, C6, C7, C8, C9: value (none) -> 100nF
- C4, C5: value (none) -> 1000uF
- Q3, Q4, Q5, Q6: value IRFI540NPBF -> IRF640
- R1, R10, R13, R14, R15, R16, R17, R35, R36, R7, R9: value (none) -> 10K
- R11, R12: value (none) -> 7,5K
- R18, R39: value (none) -> 1,2K
- R19, R21, R23, R25, R37: value (none) -> 100R
- R20, R22, R24, R26: value (none) -> 470R
- R27, R28: value (none) -> 39K
- R29, R30, R31, R32: value (none) -> 0,47R
- R3: value (none) -> 24K
- R38, R8: value (none) -> 1K
- R4: value (none) -> 13K
- R5: value (none) -> 16K
- R6: value (none) -> 2K
Other:
- note added: "FAN"
- note added: "LCD"
- note added: "Serial tag"
